Commit message: Add files via upload
Add ZED2 Camera

File: urdf/husky_ur3_gripper_old.urdf.xacro (robot description, xacro)
@@ -37,4 +37,6 @@
   <xacro:include filename="$(find rh_p12_rn_a_description)/ros2_control/rh_p12_rn_a.ros2_control.xacro" />
   -->
+  <!-- ZED Camera -->
+  <xacro:include filename="$(find husky_ur3_gripper_description)/urdf/zed_mini_macro.urdf.xacro" />
   <xacro:husky
     prefix="$(arg prefix)"
@@ -45,21 +47,28 @@
   <gazebo reference="imu_link">
     <sensor name="imu_sensor" type="imu">
+      <always_on>true</always_on>
+      <update_rate>100</update_rate>
+      <visualize>false</visualize>
+      <topic>imu</topic>  <!-- Gazebo topic -->
+      <enable_metrics>false</enable_metrics>
+      <!-- IMU plugin for Ignition Gazebo -->
       <plugin filename="libignition-gazebo-imu-system.so"
               name="ignition::gazebo::systems::Imu">
       </plugin>
+    </sensor>
+  </gazebo>
+  <gazebo reference="gps_link">
+    <sensor name="gps_sensor" type="navsat">
       <always_on>true</always_on>
-      <update_rate>100</update_rate>
-      <visualize>true</visualize>
-      <topic>imu</topic>
+      <update_rate>10</update_rate>  <!-- GPS typically 1-10 Hz -->
+      <visualize>false</visualize>
+      <topic>navsat</topic>  <!-- Gazebo topic -->
+      <!-- GPS plugin -->
+      <plugin filename="libignition-gazebo-navsat-system.so"
+              name="ignition::gazebo::systems::NavSat">
+        <frame_id>gps_link</frame_id>
+      </plugin>
     </sensor>
   </gazebo>
-  <!--
-  <gazebo reference="imu_link">
-    <sensor name="imu_sensor" type="imu">
-      <always_on>true</always_on>
-      <update_rate>100</update_rate>
-    </sensor>
-  </gazebo>
-  -->
   <!-- Connect Husky's base_link to the new mount link at the desired pose -->
   <link name="ur3_mount"/>
@@ -82,5 +91,5 @@
     generate_ros2_control_tag="false"
     >
-    <origin xyz="0 0 0" rpy="0 0 0" />
+    <origin xyz="0 0 0" rpy="0 0 ${pi}" />
   </xacro:ur_robot>
   <!-- Gripper to UR3 -->
@@ -92,4 +101,11 @@
   <xacro:rh_p12_rn_a prefix="$(arg prefix)" />
   <xacro:rh_p12_rn_a_gazebo prefix="$(arg prefix)" />
+  <!-- ZED to HUSKY -->
+  <xacro:zed_camera name="zed2" model="zed2" />
+  <joint name="zed2_mount_joint" type="fixed">
+  	<parent link="top_plate_link"/>
+  	<child  link="zed2_base_link"/>
+  	<origin xyz="0.4 0 0.1" rpy="0 0 0"/>
+  </joint>
   <!--
   <xacro:rh_p12_rn_a_system
@@ -161,4 +177,5 @@
             name="ignition::gazebo::systems::JointPositionController">
       <joint_name>ur3_shoulder_pan_joint</joint_name>
+      <topic>ur3_shoulder_pan_joint/cmd_pos</topic>
       <p_gain>500</p_gain>
       <i_gain>100</i_gain>
@@ -169,4 +186,5 @@
             name="ignition::gazebo::systems::JointPositionController">
       <joint_name>ur3_shoulder_lift_joint</joint_name>
+      <topic>ur3_shoulder_lift_joint/cmd_pos</topic>
       <p_gain>500</p_gain>
       <i_gain>100</i_gain>
@@ -177,4 +195,5 @@
             name="ignition::gazebo::systems::JointPositionController">
       <joint_name>ur3_elbow_joint</joint_name>
+      <topic>ur3_elbow_joint/cmd_pos</topic>
       <p_gain>500</p_gain>
       <i_gain>100</i_gain>
@@ -185,4 +204,5 @@
             name="ignition::gazebo::systems::JointPositionController">
       <joint_name>ur3_wrist_1_joint</joint_name>
+      <topic>ur3_wrist_1_joint/cmd_pos</topic>
       <p_gain>500</p_gain>
       <i_gain>100</i_gain>
@@ -195,4 +215,5 @@
             name="ignition::gazebo::systems::JointPositionController">
       <joint_name>ur3_wrist_2_joint</joint_name>
+      <topic>ur3_wrist_2_joint/cmd_pos</topic>
       <p_gain>500</p_gain>
       <i_gain>100</i_gain>
@@ -205,4 +226,5 @@
             name="ignition::gazebo::systems::JointPositionController">
       <joint_name>ur3_wrist_3_joint</joint_name>
+      <topic>ur3_wrist_3_joint/cmd_pos</topic>
       <p_gain>500</p_gain>
       <i_gain>100</i_gain>
